Commit message: fixa simulering

File: src/navigation_core/description/gazebo_control.xacro (robot description, xacro)
@@ -6,6 +6,6 @@
             <left_joint>left_wheel_joint</left_joint>
             <right_joint>right_wheel_joint</right_joint>
-            <wheel_separation>0.297</wheel_separation>
-            <wheel_radius>0.033</wheel_radius>
+            <wheel_separation>1</wheel_separation>
+            <wheel_radius>0.25</wheel_radius>
             <!-- Limits -->
             <!-- <max_wheel_torque>200</max_wheel_torque> -->

File: src/navigation_core/description/robot_core.xacro (robot description, xacro)
@@ -10,5 +10,5 @@
     <xacro:property name="wheel_mass" value="0.05"/>
     <xacro:property name="wheel_offset_x" value="0.25"/>
-    <xacro:property name="wheel_offset_y" value="0.45"/>
+    <xacro:property name="wheel_offset_y" value="0.5"/>
     <xacro:property name="wheel_offset_z" value="0.01"/>
     <xacro:property name="caster_wheel_radius" value="0.2"/>
